File: designs/arena_10_of_10_v1r1/layout_tool/modified_arena_10_of_10_v1r1.kicad_pcb (KiCad board)
At the start: 2 copper layers, 509 parts, among them J1 Cetus RJ45 Magjack, J10 Conn_01x05, J11 Conn_01x05, J12 Conn_01x05, J13 Conn_01x05, J14 Conn_01x05, J15 Conn_01x05, J16 Conn_01x05, J17 Conn_01x05, J18 Conn_01x05, J19 Conn_01x05, J2 Conn_01x02, J20 Conn_01x05, J21 Conn_01x05, J22 Conn_01x05, J23 Conn_01x05, J24 Conn_01x05, J25 Barrel_Jack, J26 Barrel_Jack, J27 Conn_Coaxial, J28 Conn_Coaxial, J29 Conn_Coaxial, J3 Conn_Coaxial, J4 Conn_Coaxial, J5 Conn_01x05, J6 Conn_01x05, J7 Conn_01x05, J8 Conn_01x05, J9 Conn_01x05, P1 NA, P10 NA, P2 NA, P3 NA, P4 NA, P5 NA, P6 NA, P7 NA, P8 NA, P9 NA, SW1 SW_SPDT, U1 Teensy4.1, U10 74LVC2G17, U100 74LVC1G125, U101 74LVC2G17, U102 SN74HCS08, U103 SN74HCS08, U104 74LVC1G125, U105 74LVC2G17, U106 SN74HCS08, U107 SN74HCS08, U108 74LVC1G125, U109 74LVC2G17, U11 74LVC2G17, U112 74LVC1G125, U113 74LVC2G17, U116 74LVC1G125, U117 74LVC2G17, U12 74LVC2G17, U120 74LVC1G125, U121 74LVC2G17, U124 74LVC1G125, U125 74LVC2G17, U13 74LVC2G17, U14 74LVC2G17, U15 74LVC2G17, U16 74LVC2G17, U17 74LVC2G17, U18 74LVC2G17, U19 74LVC2G17, U2 SN74LV1T34DBV, U20 74LVC2G17, U21 74LVC2G17, U22 74LVC2G17, U23 74LVC2G17, U24 74LVC2G17, U25 74LVC2G17, U26 74LVC2G17, U27 74LVC2G17, U28 74LVC2G17, U29 74LVC2G17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

Commit message: Complete initial layout of panel columns.
Finished initial config file for laying out panel columns and the
associated signal conditioning components.
Parts:
- moved U58 407.2 mm to (166.5, 97.3), turned to -72 degrees
- moved R131 404.4 mm to (168.4, 99.9), turned to -72 degrees
- moved R132 403.5 mm to (166.5, 100.6), turned to -72 degrees
- moved U59 402.1 mm to (159.4, 100.5), turned to -162 degrees
- moved C63 399.9 mm to (167.5, 100.2), turned to -72 degrees
- moved R133 396.0 mm to (156.1, 100.4), turned to -162 degrees
- moved R130 392.2 mm to (156.8, 102.4), turned to -162 degrees
- moved C64 391.1 mm to (156.5, 101.4), turned to -162 degrees
- moved J13 389.4 mm to (174.6, 101.6), turned to -72 degrees
- moved U60 385.1 mm to (139.7, 106.2), turned to -72 degrees
- moved U61 382.9 mm to (134.8, 107.7), turned to -72 degrees
- moved C62 382.8 mm to (173.3, 97.1), turned to -72 degrees
- moved R134 380.4 mm to (141.6, 108.8), turned to -72 degrees
- moved R135 379.5 mm to (139.6, 109.4), turned to -72 degrees
- moved R136 377.8 mm to (136.7, 110.4), turned to -72 degrees
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Other:
- board outline added: 228.6 x 228.6 mm
