File: designs/arena_10_of_10_v1r1/arena_10_of_10_v1r1.kicad_pcb (KiCad board)
At the start: 2 copper layers, 509 parts, among them J1 Cetus RJ45 Magjack, J10 Conn_01x05, J11 Conn_01x05, J12 Conn_01x05, J13 Conn_01x05, J14 Conn_01x05, J15 Conn_01x05, J16 Conn_01x05, J17 Conn_01x05, J18 Conn_01x05, J19 Conn_01x05, J2 Conn_01x02, J20 Conn_01x05, J21 Conn_01x05, J22 Conn_01x05, J23 Conn_01x05, J24 Conn_01x05, J25 Barrel_Jack, J26 Barrel_Jack, J27 Conn_Coaxial, J28 Conn_Coaxial, J29 Conn_Coaxial, J3 Conn_Coaxial, J4 Conn_Coaxial, J5 Conn_01x05, J6 Conn_01x05, J7 Conn_01x05, J8 Conn_01x05, J9 Conn_01x05, P1 NA, P10 NA, P2 NA, P3 NA, P4 NA, P5 NA, P6 NA, P7 NA, P8 NA, P9 NA, SW1 SW_SPDT, U1 Teensy4.1, U10 74LVC2G17, U100 74LVC1G125, U101 74LVC2G17, U102 SN74HCS08, U103 SN74HCS08, U104 74LVC1G125, U105 74LVC2G17, U106 SN74HCS08, U107 SN74HCS08, U108 74LVC1G125, U109 74LVC2G17, U11 74LVC2G17, U112 74LVC1G125, U113 74LVC2G17, U116 74LVC1G125, U117 74LVC2G17, U12 74LVC2G17, U120 74LVC1G125, U121 74LVC2G17, U124 74LVC1G125, U125 74LVC2G17, U13 74LVC2G17, U14 74LVC2G17, U15 74LVC2G17, U16 74LVC2G17, U17 74LVC2G17, U18 74LVC2G17, U19 74LVC2G17, U2 SN74LV1T34DBV, U20 74LVC2G17, U21 74LVC2G17, U22 74LVC2G17, U23 74LVC2G17, U24 74LVC2G17, U25 74LVC2G17, U26 74LVC2G17, U27 74LVC2G17, U28 74LVC2G17, U29 74LVC2G17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

Commit message: More work on layout.
Parts:
- added C130: 0.1uF, Capacitor_SMD:C_0402_1005Metric, F.Cu at (343.2, 283.7)
- added C131: 0.1uF, Capacitor_SMD:C_0402_1005Metric, F.Cu at (359.3, 283.9)
- added C132: 0.1uF, Capacitor_SMD:C_0402_1005Metric, F.Cu at (375.0, 284.4)
- added C133: 0.1uF, Capacitor_SMD:C_0402_1005Metric, F.Cu at (392.8, 284.9)
- added C134: 0.1uF, Capacitor_SMD:C_0402_1005Metric, F.Cu at (409.9, 284.4)
- added C135: 0.1uF, Capacitor_SMD:C_0402_1005Metric, F.Cu at (342.1, 304.8)
- added C136: 0.1uF, Capacitor_SMD:C_0402_1005Metric, F.Cu at (358.7, 304.9)
- added C137: 0.1uF, Capacitor_SMD:C_0402_1005Metric, F.Cu at (376.1, 304.8)
- added C138: 0.1uF, Capacitor_SMD:C_0402_1005Metric, F.Cu at (393.6, 304.8)
- added C139: 0.1uF, Capacitor_SMD:C_0402_1005Metric, F.Cu at (412.1, 304.8)
- moved U24 625.4 mm to (361.9, 232.0)
- moved R65 624.6 mm to (365.0, 233.0)
- moved R64 624.5 mm to (364.9, 230.9)
- moved C24 623.9 mm to (365.0, 232.0)
- moved C128 622.5 mm to (410.2, 295.4)
- moved R213 622.3 mm to (412.2, 306.7), turned to 180 degrees
- moved C129 622.0 mm to (405.4, 305.8)
- moved U124 621.8 mm to (409.1, 305.8)
- moved U35 621.1 mm to (370.5, 218.5)
- moved R1 620.3 mm to (308.6, 244.3), turned to -90 degrees
- moved R87 620.2 mm to (373.6, 219.5)
- moved U107 620.2 mm to (405.5, 299.2)
- moved R86 620.2 mm to (373.6, 217.5)
- moved C35 619.6 mm to (373.6, 218.5)
- moved J3 618.9 mm to (304.8, 193.0), turned to -90 degrees
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Other:
- board outline added: 248.9 x 228.6 mm
- board text added: "10-10 Teensy G6 Arena V1R1"
- board text added: "5V"
- board text added: "5V TOP"
- board text added: "ON OFF"
- board text added: "https://reiserlab.github.io/Modular-LED-Display/"

Commit message: More work on layout. Fixed header issue.
Parts:
- J10, J11, J12, J13, J14, J15, J16, J17, J18, J19, J20, J21, J22, J23, J24, J5, J6, J7, J8, J9: footprint Connector_PinHeader_2.54mm:PinHeader_1x05_P2.54mm_Vertical -> Connector_PinSocket_2.54mm:PinSocket_1x05_P2.54mm_Vertical
- moved C116 233.0 mm to (247.7, 91.3)
- moved R196 233.0 mm to (247.7, 99.0)
- moved U95 233.0 mm to (242.9, 95.2)
- moved C117 233.0 mm to (242.9, 102.0)
- moved C133 233.0 mm to (249.6, 101.1)
- moved R195 233.0 mm to (249.6, 103.0)
- moved R197 233.0 mm to (242.9, 101.0)
- moved U100 233.0 mm to (246.5, 102.0)
- moved U101 233.0 mm to (239.8, 102.0)
- moved C118 215.1 mm to (270.5, 109.5)
- moved C119 215.1 mm to (265.6, 119.9)
- moved C134 215.1 mm to (272.5, 119.0)
- moved R198 215.1 mm to (272.5, 120.9)
- moved U104 215.1 mm to (269.4, 119.9)
- moved U105 215.1 mm to (262.5, 119.9)
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
Commit message: Completed preliminary layout.
Parts:
- moved R76 121.9 mm to (252.4, 237.0), turned to 90 degrees
- moved C30 120.8 mm to (253.4, 236.9), turned to 90 degrees
- moved R77 119.7 mm to (254.4, 237.0), turned to 90 degrees
- moved R75 118.4 mm to (254.7, 270.4), turned to -90 degrees
- moved U30 118.1 mm to (253.4, 240.1), turned to 90 degrees
- moved C29 117.8 mm to (255.8, 270.4), turned to -90 degrees
- moved R74 117.3 mm to (256.8, 270.4), turned to -90 degrees
- moved U29 113.8 mm to (255.8, 267.3), turned to -90 degrees
- moved R69 110.1 mm to (266.5, 270.4), turned to -90 degrees
- moved U26 109.4 mm to (267.6, 267.3), turned to -90 degrees
- moved C26 108.7 mm to (267.6, 270.4), turned to -90 degrees
- moved R68 107.2 mm to (268.6, 270.4), turned to -90 degrees
- moved R73 103.1 mm to (262.2, 270.5), turned to -90 degrees
- moved C28 102.7 mm to (263.3, 270.5), turned to -90 degrees
- moved R72 102.2 mm to (264.3, 270.5), turned to -90 degrees
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