File: arena_12-18/fan_out.kicad_sch (KiCad schematic)
At the start: 0 parts

Commit message: starting to route
Other:
- removed sheet CIPO B1 Enable for P6
- added sheet CIPO B1 Enable for P11 (cipo_enable.kicad_sch)
Changed lines of the file:
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@@
 			(color 60 255 60 0.2)
 		)
-		(property "Sheetname" "CIPO B1 Enable for P9"
+		(property "Sheetname" "CIPO B1 Enable for P10"
 			(at 182.88 215.1884 0)
 			(show_name no)
@@
 			(color 60 255 60 0.2)
 		)
-		(property "Sheetname" "CIPO B1 Enable for P10"
+		(property "Sheetname" "CIPO B1 Enable for P11"
 			(at 229.87 215.1884 0)
 			(show_name no)
@@
 			(color 60 255 60 0.2)
 		)
-		(property "Sheetname" "CIPO B1 Enable for P8"
+		(property "Sheetname" "CIPO B1 Enable for P9"
 			(at 135.89 215.1884 0)
 			(show_name no)
@@
 			(color 60 255 60 0.2)
 		)
-		(property "Sheetname" "CIPO B1 Enable for P6"
+		(property "Sheetname" "CIPO B1 Enable for P7"
 			(at 41.91 215.1884 0)
 			(show_name no)
@@
 			(color 60 255 60 0.2)
 		)
-		(property "Sheetname" "CIPO B1 Enable for P7"
+		(property "Sheetname" "CIPO B1 Enable for P8"
 			(at 88.9 215.1884 0)
 			(show_name no)

Commit message: 1/4 left side routed
Other:
- sheet CS_03 Fan Out to P1, P7 renamed CS_03 fan out to P1, P7
Changed lines of the file:
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@@
 		)
 	)
-	(label "PAN.CS_09_P9"
+	(label "PAN.CS_09_P3"
 		(at 264.16 45.72 180)
 		(effects
@@
 		)
 	)
-	(label "PAN.CS_02_P1"
+	(label "PAN.CS_02_P7"
 		(at 200.66 58.42 180)
 		(effects
@@
 		)
 	)
-	(label "PAN.CS_16_P5"
+	(label "PAN.CS_16_P11"
 		(at 328.93 27.94 180)
 		(effects
@@
 		)
 	)
-	(label "PAN.CS_19_P11"
+	(label "PAN.CS_19_P5"
 		(at 330.2 76.2 180)
 		(effects
@@
 		)
 	)
-	(label "PAN.CS_04_P8"
+	(label "PAN.CS_04_P2"
 		(at 200.66 91.44 180)
 		(effects
@@
 		)
 	)
-	(label "PAN.CS_08_P9"
+	(label "PAN.CS_08_P3"
 		(at 264.16 30.48 180)
 		(effects
@@
 		)
 	)
-	(label "PAN.CS_23_P6"
+	(label "PAN.CS_23_P12"
 		(at 328.93 132.08 180)
 		(effects
@@
 		)
 	)
-	(label "PAN.CS_07_P8"
+	(label "PAN.CS_07_P2"
 		(at 200.66 134.62 180)
 		(effects
@@
 		)
 	)
-	(label "PAN.CS_11_P3"
+	(label "PAN.CS_11_P9"
 		(at 264.16 73.66 180)
 		(effects
@@
 		)
 	)
-	(label "PAN.CS_05_P2"
+	(label "PAN.CS_05_P8"
 		(at 200.66 104.14 180)
 		(effects
@@
 		)
 	)
-	(label "PAN.CS_22_P12"
+	(label "PAN.CS_22_P6"
 		(at 328.93 120.65 180)
 		(effects
@@
 		)
 	)
-	(label "PAN.CS_09_P3"
+	(label "PAN.CS_09_P9"
 		(at 264.16 43.18 180)
 		(effects
@@
 		)
 	)
-	(label "PAN.CS_19_P5"
+	(label "PAN.CS_17_P5"
 		(at 273.05 193.04 180)
 		(effects
@@
 		)
 	)
-	(label "PAN.CS_12_P4"
+	(label "PAN.CS_12_P10"
 		(at 264.16 88.9 180)
 		(effects
@@
 		)
 	)
-	(label "PAN.CS_20_P6"
+	(label "PAN.CS_20_P12"
 		(at 330.2 88.9 180)
 		(effects
@@
 		)
 	)
-	(label "PAN.CS_01_P1"
+	(label "PAN.CS_01_P7"
 		(at 200.66 43.18 180)
 		(effects
@@
 		)
 	)
-	(label "PAN.CS_10_P9"
+	(label "PAN.CS_10_P3"
 		(at 264.16 60.96 180)
 		(effects
@@
 		)
 	)
-	(label "PAN.CS_05_P8"
+	(label "PAN.CS_05_P2"
 		(at 200.66 106.68 180)
 		(effects
@@
 		)
 	)
-	(label "PAN.CS_00_P1"
+	(label "PAN.CS_00_P7"
 		(at 200.66 27.94 180)
 		(effects
@@
 		)
 	)
-	(label "PAN.CS_08_P3"
+	(label "PAN.CS_08_P9"
 		(at 264.16 27.94 180)
 		(effects
@@
 		)
 	)
-	(label "PAN.CS_20_P12"
+	(label "PAN.CS_20_P6"
 		(at 330.2 91.44 180)
 		(effects
@@
 		)
 	)
-	(label "PAN.CS_19_P5"
+	(label "PAN.CS_19_P11"
 		(at 330.2 73.66 180)
 		(effects
@@
 		)
 	)
-	(label "PAN.CS_17_P5"
+	(label "PAN.CS_17_P11"
 		(at 327.66 43.18 180)
 		(effects
@@
 		)
 	)
-	(label "PAN.CS_18_P11"
+	(label "PAN.CS_18_P5"
 		(at 330.2 60.96 180)
 		(effects
@@
 		)
 	)
-	(label "PAN.CS_11_P9"
+	(label "PAN.CS_11_P3"
 		(at 264.16 76.2 180)
 		(effects
@@
 		)
 	)
-	(label "PAN.CS_21_P6"
+	(label "PAN.CS_21_P12"
 		(at 328.93 102.87 180)
 		(effects
@@
 		)
 	)
-	(label "PAN.CS_21_P12"
+	(label "PAN.CS_21_P6"
 		(at 328.93 105.41 180)
 		(effects
@@
 		)
 	)
-	(label "PAN.CS_17_P5"
+	(label "PAN.CS_18_P5"
 		(at 273.05 195.58 180)
 		(effects
@@
 		)
 	)
-	(label "PAN.CS_14_P4"
+	(label "PAN.CS_14_P10"
 		(at 264.16 118.11 180)
 		(effects
@@
 		)
 	)
-	(label "PAN.CS_19_P11"
+	(label "PAN.CS_17_P11"
 		(at 273.05 220.98 180)
 		(effects
@@
 		)
 	)
-	(label "PAN.CS_04_P2"
+	(label "PAN.CS_04_P8"
 		(at 200.66 88.9 180)
 		(effects
@@
 		)
 	)
-	(label "PAN.CS_18_P5"
+	(label "PAN.CS_19_P5"
 		(at 273.05 198.12 180)
 		(effects
@@
 		)
 	)
-	(label "PAN.CS_14_P10"
+	(label "PAN.CS_14_P4"
 		(at 264.16 120.65 180)
 		(effects
@@
 		)
 	)
-	(label "PAN.CS_23_P12"
+	(label "PAN.CS_23_P6"
 		(at 328.93 134.62 180)
 		(effects
@@
 		)
 	)
-	(label "PAN.CS_02_P7"
+	(label "PAN.CS_02_P1"
 		(at 200.66 60.96 180)
 		(effects
@@
 		)
 	)
-	(label "PAN.CS_03_P7"
+	(label "PAN.CS_03_P1"
 		(at 200.66 76.2 180)
 		(effects
@@
 		)
 	)
-	(label "PAN.CS_13_P4"
+	(label "PAN.CS_13_P10"
 		(at 264.16 104.14 180)
 		(effects
@@
 		)
 	)
-	(label "PAN.CS_16_P11"
+	(label "PAN.CS_16_P5"
 		(at 328.93 30.48 180)
 		(effects
@@
 		)
 	)
-	(label "PAN.CS_03_P1"
+	(label "PAN.CS_03_P7"
 		(at 200.66 73.66 180)
 		(effects
@@
 		)
 	)
-	(label "PAN.CS_00_P7"
+	(label "PAN.CS_00_P1"
 		(at 200.66 30.48 180)
 		(effects
@@
 		)
 	)
-	(label "PAN.CS_06_P2"
+	(label "PAN.CS_06_P8"
 		(at 200.66 118.11 180)
 		(effects
@@
 		)
 	)
-	(label "PAN.CS_06_P8"
+	(label "PAN.CS_06_P2"
 		(at 200.66 120.65 180)
 		(effects
@@
 		)
 	)
-	(label "PAN.CS_18_P5"
+	(label "PAN.CS_18_P11"
 		(at 330.2 58.42 180)
 		(effects
@@
 		)
 	)
-	(label "PAN.CS_07_P2"
+	(label "PAN.CS_07_P8"
 		(at 200.66 132.08 180)
 		(effects
@@
 		)
 	)
-	(label "PAN.CS_13_P10"
+	(label "PAN.CS_13_P4"
 		(at 264.16 106.68 180)
 		(effects
@@
 		)
 	)
-	(label "PAN.CS_15_P4"
+	(label "PAN.CS_15_P10"
 		(at 264.16 132.08 180)
 		(effects
@@
 		)
 	)
-	(label "PAN.CS_15_P10"
+	(label "PAN.CS_15_P4"
 		(at 264.16 134.62 180)
 		(effects
@@
 		)
 	)
-	(label "PAN.CS_12_P10"
+	(label "PAN.CS_12_P4"
 		(at 264.16 91.44 180)
 		(effects
@@
 		)
 	)
-	(label "PAN.CS_10_P3"
+	(label "PAN.CS_10_P9"
 		(at 264.16 58.42 180)
 		(effects
@@
 		)
 	)
-	(label "PAN.CS_17_P11"
+	(label "PAN.CS_17_P5"
 		(at 327.66 45.72 180)
 		(effects
@@
 		)
 	)
-	(label "PAN.CS_22_P6"
+	(label "PAN.CS_22_P12"
 		(at 328.93 118.11 180)
 		(effects
@@
 		)
 	)
-	(label "PAN.CS_18_P11"
+	(label "PAN.CS_19_P11"
 		(at 273.05 226.06 180)
 		(effects
@@
 		)
 	)
-	(label "PAN.CS_17_P11"
+	(label "PAN.CS_18_P11"
 		(at 273.05 223.52 180)
 		(effects
@@
 		)
 	)
-	(label "PAN.CS_01_P7"
+	(label "PAN.CS_01_P1"
 		(at 200.66 45.72 180)
 		(effects
@@
 			(color 255 60 60 0.2)
 		)
-		(property "Sheetname" "CS_03 Fan Out to P1, P7"
+		(property "Sheetname" "CS_03 fan out to P1, P7"
 			(at 157.48 70.4084 0)
 			(show_name no)
