File: arena_12-18/holes.kicad_sch (KiCad schematic)
At the start: 4 parts

Commit message: 1/4 left side routed
Parts:
- added H5, H6: MountingHole_Pad, MountingHole:MountingHole_4.5mm_Pad, symbol Mechanical:MountingHole_Pad
Connections:
- net GND: now also H5.1, H6.1
