File: arena_12-18/arena_12-18.kicad_pcb (KiCad board)
At the start: 6 copper layers, 326.6 x 227.1 mm, 610 parts, among them J1 Cetus RJ45 Magjack, J10 Conn_01x05, J11 Conn_01x05, J12 Conn_01x05, J13 Conn_01x05, J14 Conn_01x05, J15 Conn_01x05, J16 Conn_01x05, J17 Conn_01x05, J18 Conn_01x05, J19 Conn_01x05, J2 Qwiic, J20 Conn_01x05, J21 Conn_01x05, J22 Conn_01x05, J23 Conn_01x05, J24 Conn_01x05, J25 Conn_01x05, J26 Conn_01x05, J27 Barrel_Jack, J28 Barrel_Jack, J29 Conn_Coaxial, J3 Conn_01x02, J30 Conn_Coaxial, J31 Conn_Coaxial, J32 Conn_01x05, J33 Conn_01x05, J34 Conn_01x05, J35 Conn_01x05, J4 Conn_01x02, J5 Conn_Coaxial, J6 Conn_Coaxial, J7 Conn_01x05, J8 Conn_01x05, J9 Conn_01x05, P1 NA, P10 NA, P11 NA, P12 NA, P2 NA, P3 NA, P4 NA, P5 NA, P6 NA, P7 NA, P8 NA, P9 NA, SW1 SW_SPDT, U1 Teensy4.1, U10 74LVC2G17, U100 74LVC1G125, U101 SN74HCS08, U102 74LVC2G17, U103 74LVC1G125, U104 SN74HCS08, U105 74LVC2G17, U106 74LVC1G125, U107 SN74HCS08, U108 74LVC2G17, U109 74LVC1G125, U11 74LVC2G17, U110 SN74HCS08, U111 74LVC2G17, U112 74LVC1G125, U113 SN74HCS08, U114 74LVC2G17, U115 74LVC1G125, U116 SN74HCS08, U117 74LVC2G17, U118 74LVC2G17, U119 74LVC2G17, U12 74LVC2G17, U120 74LVC2G17, U121 74LVC2G17, U122 74LVC1G125, U123 SN74HCS08, U124 74LVC2G17, U125 74LVC1G125, U126 SN74HCS08, U127 74LVC2G17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

Commit message: before fuses
Parts:
- added G***: LOGO, SparkFun-Qwiic:qwiic_9mm, F.Cu at (36.6, 106.2)
- U82: value RB-XXYYD -> RB-0515D
- moved C1 450.4 mm to (336.9, 140.0), turned to 180 degrees
- moved R32 447.9 mm to (340.6, 100.7), turned to 90 degrees
- moved R31 445.5 mm to (338.0, 100.7), turned to 90 degrees
- moved R11 439.7 mm to (327.8, 77.9), turned to -90 degrees
- moved R24 435.3 mm to (325.2, 98.9), turned to 90 degrees
- moved R14 426.5 mm to (315.0, 77.9), turned to -90 degrees
- moved R15 424.0 mm to (312.6, 77.9), turned to -90 degrees
- moved D2 401.5 mm to (330.4, 106.7), turned to 90 degrees
- moved D1 399.0 mm to (327.9, 102.5), turned to 90 degrees
- moved J1 365.4 mm to (343.2, 141.6), turned to 90 degrees
- moved J3 361.8 mm to (355.0, 115.0)
- moved R1 318.1 mm to (355.7, 77.9), turned to -90 degrees
- moved R2 308.0 mm to (350.6, 77.9), turned to -90 degrees
- moved R21 306.8 mm to (350.6, 98.8)
- moved R3 302.9 mm to (348.1, 77.9), turned to -90 degrees
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Routing:
- net /Fan Out/TNY.EINT: track 136.8 -> 673.3 mm, vias 2 -> 9
- net /Analog IO/I2C.SCL: track 0.00 -> 391.6 mm
- net /Fan Out/TNY.CIPO_B1: track 0.00 -> 389.5 mm, vias 0 -> 6
- net /Analog IO/I2C.SDA: track 0.00 -> 387.8 mm
- net /Fan Out/TNY.SCK_B0: track 124.4 -> 470.5 mm, vias 2 -> 5
- net /Analog IO/AIN.A0: track 0.00 -> 336.9 mm, vias 0 -> 2
- net /Fan Out/TNY.SCK_B1: track 0.00 -> 336.6 mm, vias 0 -> 6
- net /Analog IO/AIN.A1: track 0.00 -> 334.4 mm, vias 0 -> 2
- net /Fan Out/TNY.COPI_B1: track 0.00 -> 327.7 mm, vias 0 -> 4
- net /Teensy/Qwiic_SDA: track 0.00 -> 326.8 mm, vias 0 -> 3
- net /Fan Out/TNY.COPI_B0: track 125.5 -> 451.1 mm, vias 2 -> 4
- net /Teensy/Qwiic_SDL: track 0.00 -> 324.3 mm, vias 0 -> 3
- net /Teensy/D35_0_3V3: track 0.00 -> 301.2 mm, vias 0 -> 3
- net /Teensy/D29_0_3V3: track 0.00 -> 294.4 mm, vias 0 -> 3
- net Net-(U1-36_CS): track 0.00 -> 289.6 mm, vias 0 -> 3
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- added copper zone on In2.Cu, net +15V
- added copper zone on In2.Cu, net -15V
Other:
- board size 326.6 x 227.1 mm -> 330 x 240 mm
- board text added: "${ISSUE_DATE}"
- board text added: "${REVISION}"
- board text added: "${TITLE}"
- board text added: "0…5V"
- board text added: "5V → Teensy"
- board text added: "Analog Input 1 ±10V"
- board text added: "Analog Input 2 ±10V"
- board text added: "Analog Output 0…5V"
- board text added: "DIO 1"
- board text added: "DIO 2"
- board text added: "DIO2 → EINT"
