File: arena_12-18/arena_12-18.kicad_pcb (KiCad board)
At the start: 6 copper layers, 330 x 240 mm, 611 parts, among them J1 Cetus RJ45 Magjack, J10 Conn_01x05, J11 Conn_01x05, J12 Conn_01x05, J13 Conn_01x05, J14 Conn_01x05, J15 Conn_01x05, J16 Conn_01x05, J17 Conn_01x05, J18 Conn_01x05, J19 Conn_01x05, J2 Qwiic, J20 Conn_01x05, J21 Conn_01x05, J22 Conn_01x05, J23 Conn_01x05, J24 Conn_01x05, J25 Conn_01x05, J26 Conn_01x05, J27 Barrel_Jack, J28 Barrel_Jack, J29 Conn_Coaxial, J3 Conn_01x02, J30 Conn_Coaxial, J31 Conn_Coaxial, J32 Conn_01x05, J33 Conn_01x05, J34 Conn_01x05, J35 Conn_01x05, J4 Conn_01x02, J5 Conn_Coaxial, J6 Conn_Coaxial, J7 Conn_01x05, J8 Conn_01x05, J9 Conn_01x05, P1 NA, P10 NA, P11 NA, P12 NA, P2 NA, P3 NA, P4 NA, P5 NA, P6 NA, P7 NA, P8 NA, P9 NA, SW1 SW_SPDT, U1 Teensy4.1, U10 74LVC2G17, U100 74LVC1G125, U101 SN74HCS08, U102 74LVC2G17, U103 74LVC1G125, U104 SN74HCS08, U105 74LVC2G17, U106 74LVC1G125, U107 SN74HCS08, U108 74LVC2G17, U109 74LVC1G125, U11 74LVC2G17, U110 SN74HCS08, U111 74LVC2G17, U112 74LVC1G125, U113 SN74HCS08, U114 74LVC2G17, U115 74LVC1G125, U116 SN74HCS08, U117 74LVC2G17, U118 74LVC2G17, U119 74LVC2G17, U12 74LVC2G17, U120 74LVC2G17, U121 74LVC2G17, U122 74LVC1G125, U123 SN74HCS08, U124 74LVC2G17, U125 74LVC1G125, U126 SN74HCS08, U127 74LVC2G17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

Commit message: export v1.0
Parts:
- added F1: 1206L005/110WR, Fuse:Fuse_1206_3216Metric, F.Cu at (59.2, 265.4)
- added F10: 1206L005/110WR, Fuse:Fuse_1206_3216Metric, F.Cu at (334.4, 263.6)
- added F11: 1206L005/110WR, Fuse:Fuse_1206_3216Metric, F.Cu at (194.3, 102.6)
- added F12: 1206L005/110WR, Fuse:Fuse_1206_3216Metric, F.Cu at (316.2, 307.4)
- added F2: 1206L005/110WR, Fuse:Fuse_1206_3216Metric, F.Cu at (59.4, 218.8)
- added F3: 1206L005/110WR, Fuse:Fuse_1206_3216Metric, F.Cu at (75.5, 172.5)
- added F4: 1206L005/110WR, Fuse:Fuse_1206_3216Metric, F.Cu at (106.2, 135.1)
- added F5: 1206L005/110WR, Fuse:Fuse_1206_3216Metric, F.Cu at (147.9, 110.7)
- added F6: 1206L005/110WR, Fuse:Fuse_1206_3216Metric, F.Cu at (242.2, 110.9)
- added F7: 1206L005/110WR, Fuse:Fuse_1206_3216Metric, F.Cu at (285.9, 133.4)
- added F8: 1206L005/110WR, Fuse:Fuse_1206_3216Metric, F.Cu at (316.2, 170.4)
- added F9: 1206L005/110WR, Fuse:Fuse_1206_3216Metric, F.Cu at (334.1, 214.5)
- U82: value RB-0515D -> RB-XXYYD
- moved C157 2.65 mm to (317.2, 304.2)
- moved C84 2.58 mm to (329.4, 211.6)
- moved C152 2.51 mm to (190.3, 103.6)
- moved C89 2.48 mm to (331.5, 259.1)
- moved C79 2.48 mm to (311.4, 167.8)
- moved C69 2.34 mm to (237.5, 110.7)
- moved C64 2.32 mm to (144.1, 114.6)
- moved C74 2.23 mm to (279.6, 132.9)
- moved C59 2.13 mm to (104.1, 139.8)
- moved C49 1.97 mm to (60.6, 222.4)
- moved C48 1.88 mm to (62.2, 269.8)
- moved C54 1.83 mm to (75.0, 177.0)
Connections:
- C152 pad 2: +5V -> Net-(J32-Pin_1)
- C157 pad 2: +5V -> Net-(J34-Pin_1)
- C48 pad 2: +5V -> Net-(J7-Pin_1)
- C49 pad 2: +5V -> Net-(J9-Pin_1)
- C54 pad 2: +5V -> Net-(J11-Pin_1)
- C59 pad 2: +5V -> Net-(J13-Pin_1)
- C64 pad 2: +5V -> Net-(J15-Pin_1)
- C69 pad 2: +5V -> Net-(J17-Pin_1)
- C74 pad 2: +5V -> Net-(J19-Pin_1)
- C79 pad 2: +5V -> Net-(J21-Pin_1)
- C84 pad 2: +5V -> Net-(J23-Pin_1)
- C89 pad 2: +5V -> Net-(J25-Pin_1)
- J11 pad 1: +5V -> Net-(J11-Pin_1)
- J13 pad 1: +5V -> Net-(J13-Pin_1)
- J15 pad 1: +5V -> Net-(J15-Pin_1)
- J17 pad 1: +5V -> Net-(J17-Pin_1)
- J19 pad 1: +5V -> Net-(J19-Pin_1)
- J21 pad 1: +5V -> Net-(J21-Pin_1)
- J23 pad 1: +5V -> Net-(J23-Pin_1)
- J25 pad 1: +5V -> Net-(J25-Pin_1)
- J32 pad 1: +5V -> Net-(J32-Pin_1)
- J34 pad 1: +5V -> Net-(J34-Pin_1)
- J7 pad 1: +5V -> Net-(J7-Pin_1)
- J9 pad 1: +5V -> Net-(J9-Pin_1)
Routing:
- net +5V: track 131.8 -> 10.3 mm, vias 3 -> 15
- net Net-(J25-Pin_1): track 0.00 -> 11.9 mm
- net Net-(J19-Pin_1): track 0.00 -> 11.6 mm
- net Net-(J23-Pin_1): track 0.00 -> 11.5 mm
- net Net-(J21-Pin_1): track 0.00 -> 11.2 mm
- net Net-(J13-Pin_1): track 0.00 -> 10.4 mm
- net Net-(J32-Pin_1): track 0.00 -> 10.4 mm
- net Net-(J15-Pin_1): track 0.00 -> 10.2 mm
- net Net-(J7-Pin_1): track 0.00 -> 10.0 mm
- net Net-(J17-Pin_1): track 0.00 -> 9.64 mm
- net Net-(J9-Pin_1): track 0.00 -> 9.54 mm
- net Net-(J11-Pin_1): track 0.00 -> 9.28 mm
- net Net-(J34-Pin_1): track 0.00 -> 8.85 mm
- net /Analog IO/AIN.A0: track 336.9 -> 345.1 mm
- net /Analog IO/I2C.SCL: track 391.6 -> 387.0 mm
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