File: arena_12-18/arena_12-18.kicad_pcb (KiCad board)
At the start: 6 copper layers, 330 x 240 mm, 623 parts, among them J1 Cetus RJ45 Magjack, J10 Conn_01x05, J11 Conn_01x05, J12 Conn_01x05, J13 Conn_01x05, J14 Conn_01x05, J15 Conn_01x05, J16 Conn_01x05, J17 Conn_01x05, J18 Conn_01x05, J19 Conn_01x05, J2 Qwiic, J20 Conn_01x05, J21 Conn_01x05, J22 Conn_01x05, J23 Conn_01x05, J24 Conn_01x05, J25 Conn_01x05, J26 Conn_01x05, J27 Barrel_Jack, J28 Barrel_Jack, J29 Conn_Coaxial, J3 Conn_01x02, J30 Conn_Coaxial, J31 Conn_Coaxial, J32 Conn_01x05, J33 Conn_01x05, J34 Conn_01x05, J35 Conn_01x05, J4 Conn_01x02, J5 Conn_Coaxial, J6 Conn_Coaxial, J7 Conn_01x05, J8 Conn_01x05, J9 Conn_01x05, P1 NA, P10 NA, P11 NA, P12 NA, P2 NA, P3 NA, P4 NA, P5 NA, P6 NA, P7 NA, P8 NA, P9 NA, SW1 SW_SPDT, U1 Teensy4.1, U10 74LVC2G17, U100 74LVC1G125, U101 SN74HCS08, U102 74LVC2G17, U103 74LVC1G125, U104 SN74HCS08, U105 74LVC2G17, U106 74LVC1G125, U107 SN74HCS08, U108 74LVC2G17, U109 74LVC1G125, U11 74LVC2G17, U110 SN74HCS08, U111 74LVC2G17, U112 74LVC1G125, U113 SN74HCS08, U114 74LVC2G17, U115 74LVC1G125, U116 SN74HCS08, U117 74LVC2G17, U118 74LVC2G17, U119 74LVC2G17, U12 74LVC2G17, U120 74LVC2G17, U121 74LVC2G17, U122 74LVC1G125, U123 SN74HCS08, U124 74LVC2G17, U125 74LVC1G125, U126 SN74HCS08, U127 74LVC2G17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

Commit message: generate files for 12-18 G6 arena v1.0
Parts:
- U82: value RB-XXYYD -> RB-0515D
Other:
- board text added: "5V"
- board text added: "5V → Top"
- board text added: "Inner Diameter: 254mm"
- board text added: "Off"
- board text added: "On"
- board text added: "https://reiserlab.github.io/Modular-LED-Display/G6/"
Changed lines of the file:
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@@
 		(at 348 156 -90)
 		(property "Reference" "J27"
-			(at 0 4.9 270)
+			(at -6.4 -10 0)
 			(unlocked yes)
 			(layer "F.SilkS")
@@
 		(at 348 196 -90)
 		(property "Reference" "J28"
-			(at 0 4.9 270)
+			(at -6.4 -10.4 0)
 			(unlocked yes)
 			(layer "F.SilkS")
@@
 			(at 0 -6.35 90)
 			(layer "F.SilkS")
+			(hide yes)
 			(effects
 				(font
@@
 			)
 		)
-		(property "Value" "RB-XXYYD"
+		(property "Value" "RB-0515D"
 			(at 11.684 1.016 90)
 			(layer "F.SilkS")
@@
 		)
 	)
+	(gr_arc
+		(start 257.447101 86.4)
+		(mid 258.8 83.020661)
+		(end 260.312108 86.331824)
+		(stroke
+			(width 0.1)
+			(type default)
+		)
+		(layer "F.SilkS")
+	)
+	(gr_circle
+		(center 258.847101 85)
+		(end 259.647101 85)
+		(stroke
+			(width 0.1)
+			(type solid)
+		)
+		(fill yes)
+		(layer "F.SilkS")
+	)
+	(gr_line
+		(start 259.8 85)
+		(end 288.283401 85)
+		(stroke
+			(width 0.1)
+			(type default)
+		)
+		(layer "F.SilkS")
+	)
+	(gr_arc
+		(start 257.447101 86.4)
+		(mid 258.8 83.020661)
+		(end 260.312108 86.331824)
+		(stroke
+			(width 0.1)
+			(type solid)
+		)
+		(layer "B.SilkS")
+	)
+	(gr_circle
+		(center 258.847101 85)
+		(end 259.647101 85)
+		(stroke
+			(width 0.1)
+			(type solid)
+		)
+		(fill yes)
+		(layer "B.SilkS")
+	)
+	(gr_line
+		(start 259.8 85)
+		(end 288.283401 85)
+		(stroke
+			(width 0.1)
+			(type solid)
+		)
+		(layer "B.SilkS")
+	)
 	(gr_curve
 		(pts
@@
 		)
 	)
+	(gr_text "Off"
+		(at 349 168.4 90)
+		(layer "F.SilkS")
+		(effects
+			(font
+				(size 1.5 1.5)
+			)
+			(justify left bottom)
+		)
+	)
+	(gr_text "On"
+		(at 349 182.4 90)
+		(layer "F.SilkS")
+		(effects
+			(font
+				(size 1.5 1.5)
+			)
+			(justify left bottom)
+		)
+	)
+	(gr_text "5V → Top"
+		(at 345.6 201.2 90)
+		(layer "F.SilkS")
+		(effects
+			(font
+				(size 1.5 1.5)
+				(bold yes)
+			)
+			(justify left bottom)
+		)
+	)
 	(gr_text "5V → Teensy"
 		(at 353 119.6 90)
@@
 		)
 	)
+	(gr_text "Inner Diameter: 254mm"
+		(at 261.2 84.8 0)
+		(layer "F.SilkS")
+		(effects
+			(font
+				(size 1.5 1.5)
+				(thickness 0.125)
+			)
+			(justify left bottom)
+		)
+	)
 	(gr_text "Analog Output\n0…5V"
 		(at 47 195.4 0)
@@
 		)
 	)
+	(gr_text "https://reiserlab.github.io/Modular-LED-Display/G6/"
+		(at 210.6 77.6 0)
+		(layer "F.SilkS")
+		(effects
+			(font
+				(size 1.5 1.5)
+				(thickness 0.3)
+				(bold yes)
+			)
+			(justify left bottom)
+		)
+	)
 	(gr_text "${REVISION}"
 		(at 150.4 81.2 0)
@@
 		)
 	)
+	(gr_text "5V"
+		(at 345 158.4 90)
+		(layer "F.SilkS" knockout)
+		(effects
+			(font
+				(size 4 4)
+				(bold yes)
+			)
+			(justify left bottom)
+		)
+	)
 	(gr_text "DIO 1"
 		(at 47 127 0)
@@
 		)
 	)
+	(gr_text "Off"
+		(at 349 168.4 90)
+		(layer "B.SilkS")
+		(effects
+			(font
+				(size 1.5 1.5)
+			)
+			(justify right bottom mirror)
+		)
+	)
+	(gr_text "On"
+		(at 349 182.4 90)
+		(layer "B.SilkS")
+		(effects
+			(font
+				(size 1.5 1.5)
+			)
+			(justify right bottom mirror)
+		)
+	)
+	(gr_text "5V → Top"
+		(at 345.6 201.2 90)
+		(layer "B.SilkS")
+		(effects
+			(font
+				(size 1.5 1.5)
+				(bold yes)
+			)
+			(justify right bottom mirror)
+		)
+	)
+	(gr_text "Inner Diameter: 254mm"
+		(at 261.2 84.8 0)
+		(layer "B.SilkS")
+		(effects
+			(font
+				(size 1.5 1.5)
+				(thickness 0.125)
+			)
+			(justify right bottom mirror)
+		)
+	)
 	(gr_text "Analog Output\n0…5V"
 		(at 47 201.6 0)
@@
 		)
 	)
+	(gr_text "https://reiserlab.github.io/Modular-LED-Display/G6/"
+		(at 210.6 77.6 0)
+		(layer "B.SilkS")
+		(effects
+			(font
+				(size 1.5 1.5)
+				(thickness 0.3)
+				(bold yes)
+			)
+			(justify right bottom mirror)
+		)
+	)
 	(gr_text "${REVISION}"
 		(at 150.4 81.2 0)
@@
 		)
 	)
+	(gr_text "5V"
+		(at 345 158.4 90)
+		(layer "B.SilkS" knockout)
+		(effects
+			(font
+				(size 4 4)
+				(bold yes)
+			)
+			(justify right bottom mirror)
+		)
+	)
+	(barcode
+		(at 328.6 119.6 0)
+		(layer "F.SilkS")
+		(size 20 20)
+		(text "https://reiserlab.github.io/Modular-LED-Display/G6/")
+		(text_height 1.5)
+		(type qr)
+		(ecc_level M)
+		(hide yes)
+		(knockout no)
+	)
+	(barcode
+		(at 328.6 119.4 0)
+		(layer "B.SilkS")
+		(size 20 20)
+		(text "https://reiserlab.github.io/Modular-LED-Display/G6/")
+		(text_height 1.5)
+		(type qr)
+		(ecc_level M)
+		(hide yes)
+		(knockout no)
+	)
 	(segment
