File: arena_12-18/power.kicad_sch (KiCad schematic)
At the start: 4 parts, among them J27 Barrel_Jack, J28 Barrel_Jack, SW1 SW_SPDT, U82 RB-XXYYD

Commit message: generate files for 12-18 G6 arena v1.0
Parts:
- U82: value RB-XXYYD -> RB-0515D
Changed lines of the file:
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@@
 			)
 		)
-		(property "Value" "RB-XXYYD"
+		(property "Value" "RB-0515D"
 			(at 153.67 29.21 0)
 			(show_name no)
