File: arena_10-10/develop/without_reg/arena_10-10_v2r1/analog.kicad_sch (KiCad schematic)
At the start: 38 parts, among them J27 Conn_Coaxial, J28 Conn_Coaxial, J29 Conn_Coaxial, U83 OPA2277, U84 REF102AU, U85 MCP4725xxx-xCH, U86 OPA2277, U87 OPA2277

Commit message: Worked more on layout for 10 10 arena with efuse.
Parts:
- R178, R179: value 20k -> 10k; LCSC Part # C705630 -> C190095
- R180, R181: value 10k -> 20k; LCSC Part # C190095 -> C705630
Changed lines of the file:
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@@
 			)
 		)
-		(property "Value" "20k"
+		(property "Value" "10k"
 			(at 108.204 128.27 0)
 			(show_name no)
@@
 			)
 		)
-		(property "LCSC Part #" "C705630 "
+		(property "LCSC Part #" "C190095 "
 			(at 104.14 127 0)
 			(hide yes)
@@
 			)
 		)
-		(property "Value" "20k"
+		(property "Value" "10k"
 			(at 108.204 86.36 0)
 			(show_name no)
@@
 			)
 		)
-		(property "LCSC Part #" "C705630 "
+		(property "LCSC Part #" "C190095 "
 			(at 104.14 85.09 0)
 			(hide yes)
@@
 			)
 		)
-		(property "Value" "10k"
+		(property "Value" "20k"
 			(at 113.792 120.142 90)
 			(show_name no)
@@
 			)
 		)
-		(property "LCSC Part #" "C190095 "
+		(property "LCSC Part #" "C705630 "
 			(at 110.49 121.92 90)
 			(hide yes)
@@
 			)
 		)
-		(property "Value" "10k"
+		(property "Value" "20k"
 			(at 113.792 78.232 90)
 			(show_name no)
@@
 			)
 		)
-		(property "LCSC Part #" "C190095 "
+		(property "LCSC Part #" "C705630 "
 			(at 110.49 80.01 90)
 			(hide yes)
