File: arena_10-10/develop/with_reg/arena_10-10_v2r1/arena_10-10_v2r1.kicad_pcb (KiCad board)
At the start: 6 copper layers, 248.9 x 228.6 mm, 538 parts, among them J1 Cetus RJ45 Magjack, J10 Conn_01x05, J100 PinSocket_1x24_P2.54mm_Vertic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, J101 PinSocket_1x24_P2.54mm_Vertic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, J102 PinSocket_2x03_P2.00mm_Vertic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, J11 Conn_01x05, J12 Conn_01x05, J13 Conn_01x05, J14 Conn_01x05, J15 Conn_01x05, J16 Conn_01x05, J17 Conn_01x05, J18 Conn_01x05, J19 Conn_01x05, J2 Conn_01x02, J20 Conn_01x05, J21 Conn_01x05, J22 Conn_01x05, J23 Conn_01x05, J24 Conn_01x05, J25 Barrel_Jack, J26 XT30 Female, J27 Conn_Coaxial, J28 Conn_Coaxial, J29 Conn_Coaxial, J3 Conn_Coaxial, J30 Conn_01x02, J4 Conn_Coaxial, J5 Conn_01x05, J6 Conn_01x05, J7 Conn_01x05, J8 Conn_01x05, J9 Conn_01x05, P1 NA, P10 NA, P2 NA, P3 NA, P4 NA, P5 NA, P6 NA, P7 NA, P8 NA, P9 NA, SW1 SW_SPDT, U1 Teensy4.1, U10 74LVC2G17, U100 74LVC1G125, U101 74LVC2G17, U102 SN74HCS08, U103 SN74HCS08, U104 74LVC1G125, U105 74LVC2G17, U106 SN74HCS08, U107 SN74HCS08, U108 74LVC1G125, U109 74LVC2G17, U11 74LVC2G17, U110 NID100-5, U112 74LVC1G125, U113 74LVC2G17, U116 74LVC1G125, U117 74LVC2G17, U12 74LVC2G17, U120 74LVC1G125, U121 74LVC2G17, U124 74LVC1G125, U125 74LVC2G17, U13 74LVC2G17, U14 74LVC2G17, U15 74LVC2G17, U16 74LVC2G17, U17 74LVC2G17, U18 74LVC2G17, U19 74LVC2G17, U2 SN74LVC1T45DBV, U20 74LVC2G17, U21 74LVC2G17, U22 74LVC2G17, U23 74LVC2G17, U24 74LVC2G17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

Commit message: More work on zones around NID100-5 on 10-10 arena.
Routing:
- net GND: vias 283 -> 311
- net +5V: vias 23 -> 39
